File: oucrc2025-epaper.kicad_pcb (KiCad board)
At the start: 2 copper layers, 100 x 100 mm, 24 parts, among them M1 Motor_Servo, Q1 2SC2240GR, Q2 2SC2240GR, SW1 SW_Push, SW2 SW_Push, SW3 SW_Push, SW4 SW_Push

Commit message: fix: コネクタの位置を修正していなかった
Parts:
- moved M1 9.46 mm to (88.8, 90.0)
Routing:
- net +5V: track 181.2 -> 187.0 mm
- net /PWM: track 24.7 -> 22.7 mm
Changed lines of the file:
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@@
 	(footprint "Connector_PinHeader_2.54mm:PinHeader_1x03_P2.54mm_Vertical"
 		(layer "F.Cu")
-		(at 88.84 80.5)
+		(at 88.75 89.96)
 		(descr "Through hole straight pin header, 1x03, 2.54mm pitch, single row")
 		(tags "Through hole pin header THT 1x03 2.54mm single row")
@@
 	)
 	(segment
-		(start 88.84 85.58)
-		(end 93.12 89.86)
-		(width 0.4)
-		(layer "F.Cu")
-		(net 2)
-	)
-	(segment
 		(start 104.5 43.15)
 		(end 104.65 43)
@@
 	)
 	(segment
-		(start 93.12 89.86)
-		(end 96.94 89.86)
-		(width 0.4)
-		(layer "F.Cu")
-		(net 2)
-	)
-	(segment
 		(start 97.02 67)
 		(end 97.02 60.73)
@@
 	)
 	(segment
+		(start 96.94 89.86)
+		(end 91.76 95.04)
+		(width 0.4)
+		(layer "F.Cu")
+		(net 2)
+	)
+	(segment
 		(start 103.5 64.25)
 		(end 99.77 64.25)
@@
 	)
 	(segment
+		(start 91.76 95.04)
+		(end 88.75 95.04)
+		(width 0.4)
+		(layer "F.Cu")
+		(net 2)
+	)
+	(segment
 		(start 104.5 53.25)
 		(end 104.5 43.15)
@@
 	)
 	(segment
-		(start 88.84 83.04)
-		(end 88.46 83.04)
-		(width 0.2)
-		(layer "F.Cu")
-		(net 21)
-	)
-	(segment
 		(start 99.25 67.31)
-		(end 99.25 78.25)
-		(width 0.4)
-		(layer "B.Cu")
-		(net 21)
-	)
-	(segment
-		(start 94.46 83.04)
-		(end 88.84 83.04)
+		(end 99.25 82)
 		(width 0.4)
 		(layer "B.Cu")
@@
 	)
 	(segment
-		(start 99.25 78.25)
-		(end 94.46 83.04)
+		(start 99.25 82)
+		(end 88.75 92.5)
 		(width 0.4)
 		(layer "B.Cu")
@@
 	)
 	(segment
-		(start 97.25 58)
-		(end 99.56 60.31)
+		(start 99.56 67)
+		(end 99.25 67.31)
 		(width 0.4)
 		(layer "B.Cu")
@@
 	)
 	(segment
-		(start 99.56 67)
-		(end 99.25 67.31)
+		(start 97.25 58)
+		(end 99.56 60.31)
 		(width 0.4)
 		(layer "B.Cu")
@@
 	)
 	(segment
-		(start 88.84 80.5)
-		(end 100.28 80.5)
+		(start 95.25 87.75)
+		(end 93.04 89.96)
+		(width 0.3)
+		(layer "F.Cu")
+		(net 29)
+	)
+	(segment
+		(start 109.64 89.86)
+		(end 107.53 87.75)
+		(width 0.3)
+		(layer "F.Cu")
+		(net 29)
+	)
+	(segment
+		(start 107.53 87.75)
+		(end 95.25 87.75)
 		(width 0.3)
 		(layer "F.Cu")
@@
 	)
 	(segment
-		(start 100.28 80.5)
-		(end 109.64 89.86)
+		(start 93.04 89.96)
+		(end 88.75 89.96)
 		(width 0.3)
 		(layer "F.Cu")

Commit message: Add files via upload
Parts:
- renumbered SW1 to SW-A, SW2 to SW-B, SW4 to SW-L, SW3 to SW-R
Changed lines of the file:
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@@
 		(descr "Generic 6mm SW tactile push button")
 		(tags "tact sw push 6mm")
-		(property "Reference" "SW2"
+		(property "Reference" "SW-B"
 			(at 3.25 -2 0)
 			(layer "F.SilkS")
@@
 		(descr "Generic 6mm SW tactile push button")
 		(tags "tact sw push 6mm")
-		(property "Reference" "SW4"
+		(property "Reference" "SW-L"
 			(at 3.25 -2 0)
 			(layer "F.SilkS")
@@
 		(descr "Generic 6mm SW tactile push button")
 		(tags "tact sw push 6mm")
-		(property "Reference" "SW3"
+		(property "Reference" "SW-R"
 			(at 3.25 -2 0)
 			(layer "F.SilkS")
@@
 		(descr "Generic 6mm SW tactile push button")
 		(tags "tact sw push 6mm")
-		(property "Reference" "SW1"
+		(property "Reference" "SW-A"
 			(at 3.25 -2 0)
 			(layer "F.SilkS")
