File: oucrc2025-epaper.kicad_sch (KiCad schematic)
At the start: 22 parts, among them M1 Motor_Servo, Q1 2SC2240GR, Q2 2SC2240GR, SW1 SW_Push, SW2 SW_Push, SW3 SW_Push, SW4 SW_Push

Commit message: Add files via upload
Parts:
- renumbered SW1 to SW-A, SW2 to SW-B, SW4 to SW-L, SW3 to SW-R
Changed lines of the file:
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@@
 		(on_board yes)
 		(dnp no)
-		(property "Reference" "SW4"
+		(property "Reference" "SW-L"
 			(at 266.7 102.362 0)
 			(effects
@@
 			(project "OUCRC-TeamB"
 				(path "/fdd8752d-23db-4ccf-bf63-6ba6f7291126"
-					(reference "SW4")
+					(reference "SW-L")
 					(unit 1)
 				)
@@
 		(on_board yes)
 		(dnp no)
-		(property "Reference" "SW2"
+		(property "Reference" "SW-B"
 			(at 210.82 102.362 0)
 			(effects
@@
 			(project "OUCRC-TeamB"
 				(path "/fdd8752d-23db-4ccf-bf63-6ba6f7291126"
-					(reference "SW2")
+					(reference "SW-B")
 					(unit 1)
 				)
@@
 		(on_board yes)
 		(dnp no)
-		(property "Reference" "SW1"
+		(property "Reference" "SW-A"
 			(at 182.88 102.362 0)
 			(effects
@@
 			(project "OUCRC-TeamB"
 				(path "/fdd8752d-23db-4ccf-bf63-6ba6f7291126"
-					(reference "SW1")
+					(reference "SW-A")
 					(unit 1)
 				)
@@
 		(on_board yes)
 		(dnp no)
-		(property "Reference" "SW3"
+		(property "Reference" "SW-R"
 			(at 238.76 102.362 0)
 			(effects
@@
 			(project "OUCRC-TeamB"
 				(path "/fdd8752d-23db-4ccf-bf63-6ba6f7291126"
-					(reference "SW3")
-					(unit 1)
-				)
+					(reference "SW-R")
+					(unit 1)
+				)
